File: Debugger.kicad_sch (KiCad schematic)
At the start: 34 parts, among them SW3 1TS028A-1900-0600-CT, U8 HPM5301IEG1, Y2 24M

Commit message: update: 更新PCB
Parts:
- added J6: Header 2.54 4P, Connector_PinHeader_2.54mm:PinHeader_1x04_P2.54mm_Vertical, symbol Connector_Generic:Conn_01x04
Connections:
- net +3V3: now also J6.1 (Pin_1)
- net BOOT0: no longer D3.4 (DIN)
- net GND: now also J6.4 (Pin_4)
- net ISP_RX: now also J6.3 (Pin_3)
- net ISP_TX: now also J6.2 (Pin_2)
- net WS2812: now reaches U8.46 (PA07/TMR0.COMP0/URT1.TXD/I2C1.SCL/SPI0.MOSI/TRGM0.P07/JTAG.TMS)
- net WS2812: now also D3.4 (DIN)
- no-connect marks 13 -> 12
