File: HSDevKit5301.kicad_pcb (KiCad board)
At the start: 2 copper layers, 65 x 30 mm, 145 parts, among them J1 USB_C_Receptacle_USB2.0, J2 USB_C_Receptacle_USB2.0, J3 Header 2.54 2x20, J4 FH34SRJ-8S-0.5SH, J5 Micro_SD_Card_Det1, Q1 2N7002, Q2 2N7002, Q3 AO3400, Q4 AO3401A, SW1 TS3425, SW2 TS3425, SW3 1TS028A-1900-0600-CT, U1 HPM5301IEG1, U2 TPS25200, U3 0524P, U4 0524P, U5 TPS25200, U6 HUSB320, U7 RT8010, U8 HPM5301IEG1, U9 W25Q32JVSS, Y1 24M, Y2 24M

Commit message: update: 更新PCB
Parts:
- added D4: LED_R, LED_SMD:LED_0402_1005Metric, F.Cu at (28.1, 25.8)
- added D5: LED_G, LED_SMD:LED_0402_1005Metric, F.Cu at (28.1, 26.8)
- added J6: Header 2.54 4P, Connector_PinHeader_2.54mm:PinHeader_1x04_P2.54mm_Vertical, F.Cu at (90.1, 29.4)
- added R53: 10k, Resistor_SMD:R_0402_1005Metric, F.Cu at (28.1, 24.8)
- added R54: 10k, Resistor_SMD:R_0402_1005Metric, F.Cu at (30.0, 28.0)
- added R55: 0R, Resistor_SMD:R_0402_1005Metric, B.Cu at (52.0, 43.1)
- C19, C20, C22, C23, C27, C28, C32, C33, C36, C39, C44, C45, C46, C47, C48, C49, C51, C52, C53, C59, R1, R17, R2, R22, R3, R4, R40, R41, R42, R43, R44, R45, R46, R47, R48, R49, R5, R50, R51, R52, R7, R8, R9: moved to B.Cu
- Q1: footprint Package_TO_SOT_SMD:SOT-23 -> Package_TO_SOT_SMD:SOT-323_SC-70; moved to B.Cu
- Q2: footprint Package_TO_SOT_SMD:SOT-23 -> Package_TO_SOT_SMD:SOT-323_SC-70
- Q3: value AO3400 -> 2N7002; footprint Package_TO_SOT_SMD:SOT-23 -> Package_TO_SOT_SMD:SOT-323_SC-70
- R24, R25: value 0R -> 900k; moved to B.Cu
- R35: value 47k -> 10k
- R6: value 0R -> 22R; moved to B.Cu
- moved C15 81.0 mm to (44.5, 25.8), turned to -90 degrees
- moved C40 80.1 mm to (54.7, 25.8), turned to -90 degrees
- moved C28 77.1 mm to (41.4, 30.5), turned to 180 degrees
- moved R32 75.9 mm to (61.7, 25.6), turned to -90 degrees
- moved C39 75.2 mm to (62.4, 30.8)
- moved C38 75.0 mm to (57.6, 27.7), turned to 90 degrees
- moved C13 74.7 mm to (47.3, 27.7), turned to 90 degrees
- moved R31 74.3 mm to (64.6, 25.6), turned to 90 degrees
- moved C22 73.4 mm to (41.4, 35.4), turned to 180 degrees
- moved C18 73.3 mm to (47.3, 25.8), turned to -90 degrees
- moved C12 72.9 mm to (46.4, 27.7), turned to 90 degrees
- moved U8 72.9 mm to (57.0, 33.2), turned to 180 degrees
- moved C37 72.9 mm to (56.6, 27.7), turned to 90 degrees
- moved C14 72.6 mm to (52.0, 30.9)
- moved C57 72.5 mm to (62.6, 25.6), turned to 90 degrees
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Connections:
- C6 pad 1: Net-(D1-A) -> /Interface/VBUS
- D1 pad 2: Net-(D1-A) -> /Interface/VBUS
- D3 pad 4: /Debugger/BOOT0 -> /Debugger/WS2812
- J2 pad A4: Net-(D1-A) -> /Interface/VBUS
- J2 pad A9: Net-(D1-A) -> /Interface/VBUS
- J2 pad B4: Net-(D1-A) -> /Interface/VBUS
- J2 pad B9: Net-(D1-A) -> /Interface/VBUS
- J4 pad 1: unconnected-(J4-Pin_1-Pad1) -> /LCD_CS
- J4 pad 3: unconnected-(J4-Pin_3-Pad3) -> /LCD_SCK
- J4 pad 4: unconnected-(J4-Pin_4-Pad4) -> /LCD_MOSI
- J4 pad 5: unconnected-(J4-Pin_5-Pad5) -> /LCD_DC
- J4 pad 6: unconnected-(J4-Pin_6-Pad6) -> /LCD_RST
- J5 pad 8: /SD_DET -> unconnected-(J5-DAT1-Pad8)
- J5 pad 9: GND -> /SD_DET
- Q1 pad 1: Net-(Q1-G) -> /Debugger/SRST
- Q1 pad 3: /NRST -> Net-(Q1-D)
- R16 pad 2: /PY01 -> Net-(U5-~{FAULT})
- R23 pad 1: VBUS -> /Interface/VBUS
- R24 pad 1: Net-(U6-ADDR) -> Net-(U6-PORT)
- R24 pad 2: +3V3 -> GND
- R25 pad 1: Net-(U6-ADDR) -> Net-(U6-PORT)
- R25 pad 2: GND -> +3V3
- R45 pad 1: /PA10 -> /PB09
- R48 pad 1: /PB14 -> /PB15
- R49 pad 1: /PB15 -> /PB14
- R6 pad 1: Net-(Q1-G) -> /NRST
- R6 pad 2: /Debugger/SRST -> Net-(Q1-D)
- R7 pad 1: Net-(Q1-G) -> /Debugger/SRST
- U3 pad 1: /Interface/USB_D+ -> /Interface/USB_D-
- U3 pad 10: /Interface/USB_D+ -> /Interface/USB_D-
- U3 pad 2: /Interface/USB_D- -> /Interface/USB_D+
- U3 pad 9: /Interface/USB_D- -> /Interface/USB_D+
- U4 pad 1: /PA24 -> /PA25
- U4 pad 10: /PA24 -> /PA25
- U4 pad 2: /PA25 -> /PA24
- U4 pad 9: /PA25 -> /PA24
- U5 pad 1: Net-(D1-A) -> /Interface/VBUS
- U5 pad 3: /PY01 -> Net-(U5-~{FAULT})
- U6 pad 3: unconnected-(U6-PORT-Pad3) -> Net-(U6-PORT)
- U6 pad 5: Net-(U6-ADDR) -> unconnected-(U6-ADDR-Pad5)
- U8 pad 46: unconnected-(U8B-PA07/TMR0.COMP0/URT1.TXD/I2C1.SCL/SPI0.MOSI/TRGM0.P07/JTAG.TMS-Pad46) -> /Debugger/WS2812
Routing:
- net +3V3: track 0.00 -> 316.6 mm, vias 0 -> 26
- net +5V: track 0.00 -> 70.8 mm, vias 0 -> 8
- net GND: track 0.00 -> 66.8 mm, vias 0 -> 70
- net /PA26: track 0.00 -> 60.8 mm, vias 0 -> 2
- net /PA31: track 0.00 -> 60.8 mm, vias 0 -> 1
- net /PA27: track 0.00 -> 59.4 mm, vias 0 -> 2
- net /PA29: track 0.00 -> 58.9 mm, vias 0 -> 1
- net /PA28: track 0.00 -> 58.2 mm, vias 0 -> 2
- net /PB13: track 0.00 -> 57.4 mm, vias 0 -> 4
- net /PB09: track 0.00 -> 54.2 mm, vias 0 -> 1
- net /PB08: track 0.00 -> 48.8 mm
- net /PA10: track 0.00 -> 48.2 mm, vias 0 -> 3
- net VDD_SOC1: track 0.00 -> 47.9 mm, vias 0 -> 8
- net VDD_SOC0: track 0.00 -> 47.6 mm, vias 0 -> 7
- net /PY01: track 0.00 -> 45.7 mm, vias 0 -> 1
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- added copper zone on B.Cu, net GND
- added copper zone on F.Cu, net GND
- added copper zone on In1.Cu, net GND
Other:
- outline, holes or cut-outs redrawn
- copper layers 2 -> 4
- board text added: "+5V"
- board text added: "3V3"
- board text added: "D"
- board text added: "DRP(NC)"
- board text added: "GND"
- board text added: "Hpmicro Solution DevKit 5301"
- board text added: "L(A10)"
- board text added: "LCD_BL"
- board text added: "LCD_CS"
- board text added: "LCD_DC"
- board text added: "LCD_RST"
- board text added: "LCD_SCK"
- board text added: "LCD_SDA"
- board text added: "PA00"
- board text added: "PA01"
- board text added: "PA02"
- board text added: "PA03"
- board text added: "PA04"
- board text added: "PA05"
- board text added: "PA06"
- board text added: "PA07"
- board text added: "PA08"
- board text added: "PA09"
- board text added: "PA10"
- board text added: "PA26"
- board text added: "PA27"
- board text added: "PA28"
- board text added: "PA29"
- board text added: "PA30"
- board text added: "PA31"
- board text added: "PB08"
- board text added: "PB09"
- board text added: "PB10"
- board text added: "PB11"
- board text added: "PB12"
- board text added: "PB13"
- board text added: "PB14"
- board text added: "PB15"
- board text added: "PY00"
- board text added: "PY01"
- board text added: "Paste"
- board text added: "Power"
- board text added: "QSPI_CS"
- board text added: "QSPI_DAT2"
- board text added: "QSPI_DAT3"
- board text added: "QSPI_MISO"
- board text added: "QSPI_MOSI"
- board text added: "QSPI_SCLK"
- board text added: "RESRT"
- board text added: "RST"
- board text added: "RX"
- board text added: "SD_DET"
- board text added: "Sink"
- board text added: "Source"
- board text added: "TCK"
- board text added: "TDI"
- board text added: "TDO"
- board text added: "TMS"
- board text added: "TRST"
- board text added: "TX"
- board text added: "URX"
- board text added: "USB0_ID"
- board text added: "USB0_OC"
- board text added: "USB0_PWR"
- board text added: "USER"
- board text added: "UTX"
- board text added: "WK"
- board text removed: "PoE"
