File: HSDevKit5301.kicad_sch (KiCad schematic)
At the start: 48 parts, among them J4 FH34SRJ-8S-0.5SH, J5 Micro_SD_Card_Det1, Q1 2N7002, Q3 AO3400, Q4 AO3401A, SW1 TS3425, SW2 TS3425, U1 HPM5301IEG1, U9 W25Q32JVSS, Y1 24M

Commit message: update: 更新PCB
Parts:
- added D4: LED_R, LED_SMD:LED_0402_1005Metric, symbol Device:LED
- added D5: LED_G, LED_SMD:LED_0402_1005Metric, symbol Device:LED
- added R53, R54: 10k, Resistor_SMD:R_0402_1005Metric, symbol Device:R
- Q1: footprint Package_TO_SOT_SMD:SOT-23 -> Package_TO_SOT_SMD:SOT-323_SC-70
- Q3: value AO3400 -> 2N7002; footprint Package_TO_SOT_SMD:SOT-23 -> Package_TO_SOT_SMD:SOT-323_SC-70
- R35: value 47k -> 10k
- R6: value 0R -> 22R
Connections:
- net +3V3: now also R53.1, R54.1
- net Debugger/SRST: now also Q1.1 (G), R7.1; no longer R6.2
- net GND: now also D4.1 (K); no longer J5.9 (DET)
- net LCD_CS: now also J4.1 (Pin_1)
- net LCD_DC: now also J4.5 (Pin_5)
- net LCD_MOSI: now also J4.4 (Pin_4)
- net LCD_RST: now also J4.6 (Pin_6)
- net LCD_SCK: now also J4.3 (Pin_3)
- net NRST: now also R6.1; no longer Q1.3 (D)
- net PA10: now also D5.1 (K); no longer R45.1
- net PB09: now also R45.1
- net PB14: now also R49.1; no longer R48.1
- net PB15: now also R48.1; no longer R49.1
- net SD_DET: now also J5.9 (DET); no longer J5.8 (DAT1)
- new net: Q1.3 (D), R6.2
- new net: D4.2 (A), R53.2
- new net: D5.2 (A), R54.2
- no-connect marks 2 -> 3
