File: Interface.kicad_sch (KiCad schematic)
At the start: 29 parts, among them J1 USB_C_Receptacle_USB2.0, J2 USB_C_Receptacle_USB2.0, J3 Header 2.54 2x20, Q2 2N7002, U2 TPS25200, U3 0524P, U4 0524P, U5 TPS25200, U6 HUSB320

Commit message: update: 更新PCB
Parts:
- added R55: 0R, Resistor_SMD:R_0402_1005Metric, symbol Device:R
- Q2: footprint Package_TO_SOT_SMD:SOT-23 -> Package_TO_SOT_SMD:SOT-323_SC-70
- R24, R25: value 0R -> 900k
Connections:
- net +3V3: now also R25.2; no longer R24.2
- net GND: now also R24.2; no longer R25.2
- net OTG_USB_D+: now also U4.2 (D1-), U4.9 (NC); no longer U4.1 (D1+), U4.10 (NC)
- net OTG_USB_D-: now also U4.1 (D1+), U4.10 (NC); no longer U4.2 (D1-), U4.9 (NC)
- net USB0_OC: now also R55.1; no longer R16.2, U5.3 (~{FAULT})
- net USB_D+: now also U3.2 (D1-), U3.9 (NC); no longer U3.1 (D1+), U3.10 (NC)
- net USB_D-: now also U3.1 (D1+), U3.10 (NC); no longer U3.2 (D1-), U3.9 (NC)
- net VBUS: now also C6.1, D1.2 (A), J2.A4 (VBUS), J2.A9 (VBUS), J2.B4 (VBUS), J2.B9 (VBUS), U5.1 (OUT)
- net at U6.3 (PORT): now also R24.1, R25.1
- new net: R16.2, R55.2, U5.3 (~{FAULT})
- now unconnected: U6.5 (ADDR)
